File: schematic.sch (EAGLE design)
At the start: 3 parts, among them IC1 MEGA8-AI

Commit message: Added LED and STM32
Parts:
- removed IC1: MEGA8-AI, atmel:MEGA8-AI
- added C1, C2, C3, C4, C5: (no value), resistor:C-EUC0805
- added C6: (no value), resistor:CPOL-EU153CLV-0605
- added JP1: (no value), PLL:PINHD-1X8
- added R1, R2, R4, R5, R7: (no value), resistor:R-EU_R0805
- added U$3, U$4, U$5: IT1188E, misc:IT1188E
- added U$6: GL5537, misc:GL5537
- added U$7: STM32F103C8, stm32:STM32F103C8
- U$1: value MAX7219CWG -> LBT8402BW; device max7219:MAX7219CWG -> lbt8402:LBT8402BW
Connections:
- new net +5V: C6.+
- new net N$2: JP1.3, U$7.JTCK/SWCLK
- new net N$3: JP1.4, U$7.JTDI
- new net N$5: JP1.6, U$7.JNTRST
- new net PHOTO_SENSOR: C5.1, R7.2, U$6.P$1
- new net SQW: R4.1, U$2.32KHZ
- new net TIMER_INT: R5.1, U$2.INT
- net GND: now also C1.2, C2.2, C3.2, C4.2, C5.2, C6.-, R7.1, U$7.AGND, U$7.GND@1, U$7.GND@2, U$7.GND@3; no longer IC1.GND, IC1.GND@1, IC1.GND@2, U$1.GND@1, U$1.GND@2
- net N$1: now also JP1.2, U$7.JTMS/SWDIO; no longer U$2.INT
- net N$4: now also JP1.5, U$7.JTDO; no longer U$2.32KHZ
- net RST: no longer IC1.PC6(/RESET)
- net SCL: now also R2.1; no longer IC1.PC5(ADC5/SCL)
- net SDA: now also R1.1; no longer IC1.PC4(ADC4/SDA)
- net VCC: now also C1.1, C2.1, C3.1, C4.1, R1.2, R2.2, R4.2, R5.2, U$6.P$2; no longer IC1.AREF, IC1.AVCC, IC1.VCC@1, IC1.VCC@2, U$1.VCC

Commit message: .
Parts:
- removed JP1: (no value), PLL:PINHD-1X8
- added IC1: MEGA8-AI, atmel:MEGA8-AI
- added R3: (no value), resistor:R-EU_R0805
- added U$8: MICRO-USB, microusb:MICRO-USB
- added U$9: PINHD-1X5, PLL:PINHD-1X5
- U$7: value STM32F103C8 -> MAX7219CWG; device stm32:STM32F103C8 -> max7219:MAX7219CWG
Connections:
- removed net +5V: C6.+
- removed net RST: U$2.RST
- new net DIG_1: U$1.DIG_1, U$7.SEGA
- new net DSP_CLK: U$7.CLK
- new net DSP_DIN: U$7.DIN
- new net DSP_LOAD: U$7.LOAD
- new net MISO: IC1.PB4(MISO), U$9.2
- new net MOSI: IC1.PB3(MOSI/OC2), U$9.1
- new net N$10: U$1.SEG_E, U$7.DIG4
- new net N$11: U$1.SEG_F, U$7.DIG5
- new net N$12: U$1.SEG_G, U$7.DIG6
- new net N$13: U$1.DOTS_CATHODE, U$1.SEG_DOT, U$7.DIG7
- new net N$6: U$1.SEG_A, U$7.DIG0
- new net N$7: U$1.SEG_B, U$7.DIG1
- new net N$8: U$1.SEG_C, U$7.DIG2
- new net N$9: U$1.SEG_D, U$7.DIG3
- new net RESET: IC1.PC6(/RESET), U$2.RST, U$9.4
- new net SCK: IC1.PB5(SCK), U$9.3
- net GND: now also IC1.GND, IC1.GND@1, IC1.GND@2, U$8.GND@1, U$8.GND@2, U$9.5; no longer U$7.AGND, U$7.GND@3
- net N$1: now also R3.2, U$7.ISET; no longer JP1.2, U$7.JTMS/SWDIO
- net N$2: now also U$1.DIG_2, U$7.SEGB; no longer JP1.3, U$7.JTCK/SWCLK
- net N$3: now also U$1.DIG_3, U$7.SEGC; no longer JP1.4, U$7.JTDI
- net N$4: now also U$1.DIG_4, U$7.SEGD; no longer JP1.5, U$7.JTDO
- net N$5: now also U$1.DOTS_ANODE, U$7.SEGE; no longer JP1.6, U$7.JNTRST
- net SCL: now also IC1.PC5(ADC5/SCL)
- net SDA: now also IC1.PC4(ADC4/SDA)
- net VCC: now also C6.+, IC1.AREF, IC1.AVCC, IC1.VCC@1, IC1.VCC@2, R3.1, U$7.VCC
Other:
- moved on the sheet: C1, C2, C3, C4, C5, C6, R1, R2, R4, R5, R7, U$6

Commit message: .
Parts:
- added R6, R8, R9: (no value), resistor:R-EU_R0805
Connections:
- new net BTN_1: R6.1, U$3.4
- new net BTN_2: R8.1, U$4.4
- new net BTN_3: R9.1, U$5.4
- net GND: now also U$3.3, U$4.3, U$5.3
- net VCC: now also R6.2, R8.2, R9.2
Other:
- moved on the sheet: C1, C2, C3, C4, C5, C6, R3, R7, U$6, U$7, U$9

Commit message: Element placement
Parts:
- removed C6: (no value), resistor:CPOL-EU153CLV-0605
- removed R9: (no value), resistor:R-EU_R0805
- removed U$5: IT1188E, misc:IT1188E
- added B1: BATTERY1220, Battery&Holder:BATTERY1220
Connections:
- removed net BTN_3: R9.1, U$5.4
- new net N$14: B1.+, U$2.VBAT
- net BTN_1: now also IC1.PC1(ADC1)
- net BTN_2: now also IC1.PC2(ADC2)
- net DSP_CLK: now also IC1.PB0(ICP)
- net DSP_DIN: now also IC1.PB2(SS/OC1B)
- net DSP_LOAD: now also IC1.PB1(OC1A)
- net GND: now also B1.-; no longer C6.-, U$5.3
- net PHOTO_SENSOR: now also IC1.PC0(ADC0)
- net SQW: now also IC1.PD2(INT0)
- net TIMER_INT: now also IC1.PD3(INT1)
- net VCC: no longer C6.+, R9.2
Changed lines of the file:
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@@
 <part name="U$6" library="misc" deviceset="GL5537" device=""/>
 <part name="U$1" library="lbt8402" deviceset="LBT8402BW" device=""/>
-<part name="C6" library="resistor" deviceset="CPOL-EU" device="153CLV-0605"/>
 <part name="U$7" library="max7219" deviceset="MAX7219CWG" device=""/>
 <part name="GND1" library="supply1" deviceset="GND" device=""/>
@@
 <part name="R6" library="resistor" deviceset="R-EU_" device="R0805"/>
 <part name="R8" library="resistor" deviceset="R-EU_" device="R0805"/>
-<part name="R9" library="resistor" deviceset="R-EU_" device="R0805"/>
 <part name="P+11" library="supply1" deviceset="VCC" device=""/>
 <part name="U$3" library="misc" deviceset="IT1188E" device=""/>
 <part name="GND13" library="supply1" deviceset="GND" device=""/>
 <part name="U$4" library="misc" deviceset="IT1188E" device=""/>
-<part name="U$5" library="misc" deviceset="IT1188E" device=""/>
 <part name="GND14" library="supply1" deviceset="GND" device=""/>
-<part name="GND15" library="supply1" deviceset="GND" device=""/>
+<part name="B1" library="Battery&amp;Holder" deviceset="BATTERY" device="1220"/>
+<part name="GND4" library="supply1" deviceset="GND" device=""/>
 </parts>
 <sheets>
@@
 <instance part="U$6" gate="G$1" x="-43.18" y="-111.76" rot="R90"/>
 <instance part="U$1" gate="G$1" x="93.98" y="-165.1"/>
-<instance part="C6" gate="G$1" x="-43.18" y="-81.28"/>
 <instance part="U$7" gate="G$1" x="48.26" y="-121.92"/>
 <instance part="GND1" gate="1" x="27.94" y="-144.78"/>
@@
 <instance part="R6" gate="G$1" x="-43.18" y="-154.94" rot="R90"/>
 <instance part="R8" gate="G$1" x="-30.48" y="-154.94" rot="R90"/>
-<instance part="R9" gate="G$1" x="-17.78" y="-154.94" rot="R90"/>
 <instance part="P+11" gate="VCC" x="-43.18" y="-144.78"/>
 <instance part="U$3" gate="G$1" x="-45.72" y="-165.1" rot="R90"/>
 <instance part="GND13" gate="1" x="-43.18" y="-175.26"/>
 <instance part="U$4" gate="G$1" x="-33.02" y="-165.1" rot="R90"/>
-<instance part="U$5" gate="G$1" x="-20.32" y="-165.1" rot="R90"/>
 <instance part="GND14" gate="1" x="-30.48" y="-175.26"/>
-<instance part="GND15" gate="1" x="-17.78" y="-175.26"/>
+<instance part="B1" gate="2477" x="167.64" y="-35.56"/>
+<instance part="GND4" gate="1" x="167.64" y="-45.72"/>
 </instances>
 <busses>
@@
 <junction x="-27.94" y="-86.36"/>
 <wire x1="-27.94" y1="-86.36" x2="-22.86" y2="-86.36" width="0.1524" layer="91"/>
-<pinref part="C6" gate="G$1" pin="-"/>
 <wire x1="-38.1" y1="-86.36" x2="-43.18" y2="-86.36" width="0.1524" layer="91"/>
 <wire x1="-38.1" y1="-86.36" x2="-38.1" y2="-88.9" width="0.1524" layer="91"/>
@@
 </segment>
 <segment>
-<pinref part="U$5" gate="G$1" pin="3"/>
-<pinref part="GND15" gate="1" pin="GND"/>
-<wire x1="-17.78" y1="-172.72" x2="-17.78" y2="-170.18" width="0.1524" layer="91"/>
+<pinref part="B1" gate="2477" pin="-"/>
+<pinref part="GND4" gate="1" pin="GND"/>
+<wire x1="167.64" y1="-43.18" x2="167.64" y2="-40.64" width="0.1524" layer="91"/>
 </segment>
 </net>
@@
 <segment>
 <wire x1="-43.18" y1="-73.66" x2="-43.18" y2="-76.2" width="0.1524" layer="91"/>
-<pinref part="C6" gate="G$1" pin="+"/>
 <pinref part="P+1" gate="VCC" pin="VCC"/>
 <pinref part="C1" gate="G$1" pin="1"/>
@@
 </segment>
 <segment>
-<pinref part="R9" gate="G$1" pin="2"/>
 <pinref part="R6" gate="G$1" pin="2"/>
-<wire x1="-17.78" y1="-149.86" x2="-30.48" y2="-149.86" width="0.1524" layer="91"/>
 <wire x1="-30.48" y1="-149.86" x2="-43.18" y2="-149.86" width="0.1524" layer="91"/>
 <wire x1="-43.18" y1="-149.86" x2="-43.18" y2="-147.32" width="0.1524" layer="91"/>
@@
 <junction x="-43.18" y="-149.86"/>
 <pinref part="R8" gate="G$1" pin="2"/>
-<junction x="-30.48" y="-149.86"/>
 </segment>
 </net>
@@
 <label x="205.74" y="-17.78" size="1.778" layer="95"/>
 </segment>
+<segment>
+<pinref part="IC1" gate="G$1" pin="PD2(INT0)"/>
+<wire x1="76.2" y1="-35.56" x2="81.28" y2="-35.56" width="0.1524" layer="91"/>
+<label x="81.28" y="-35.56" size="1.778" layer="95"/>
+</segment>
 </net>
 <net name="TIMER_INT" class="0">
@@
 <wire x1="215.9" y1="-12.7" x2="215.9" y2="-15.24" width="0.1524" layer="91"/>
 <label x="215.9" y="-17.78" size="1.778" layer="95"/>
+</segment>
+<segment>
+<pinref part="IC1" gate="G$1" pin="PD3(INT1)"/>
+<wire x1="76.2" y1="-38.1" x2="81.28" y2="-38.1" width="0.1524" layer="91"/>
+<label x="81.28" y="-38.1" size="1.778" layer="95"/>
 </segment>
 </net>
@@
 <junction x="-43.18" y="-119.38"/>
 </segment>
+<segment>
+<pinref part="IC1" gate="G$1" pin="PC0(ADC0)"/>
+<wire x1="76.2" y1="-7.62" x2="81.28" y2="-7.62" width="0.1524" layer="91"/>
+<label x="81.28" y="-7.62" size="1.778" layer="95"/>
+</segment>
 </net>
 <net name="DIG_1" class="0">
@@
 <label x="20.32" y="-104.14" size="1.778" layer="95"/>
 </segment>
+<segment>
+<pinref part="IC1" gate="G$1" pin="PB0(ICP)"/>
+<wire x1="76.2" y1="-53.34" x2="81.28" y2="-53.34" width="0.1524" layer="91"/>
+<label x="81.28" y="-53.34" size="1.778" layer="95"/>
+</segment>
 </net>
 <net name="DSP_LOAD" class="0">
@@
 <label x="20.32" y="-109.22" size="1.778" layer="95"/>
 </segment>
+<segment>
+<pinref part="IC1" gate="G$1" pin="PB1(OC1A)"/>
+<wire x1="76.2" y1="-55.88" x2="81.28" y2="-55.88" width="0.1524" layer="91"/>
+<label x="81.28" y="-55.88" size="1.778" layer="95"/>
+</segment>
 </net>
 <net name="DSP_DIN" class="0">
@@
 <wire x1="33.02" y1="-114.3" x2="20.32" y2="-114.3" width="0.1524" layer="91"/>
 <label x="20.32" y="-114.3" size="1.778" layer="95"/>
+</segment>
+<segment>
+<pinref part="IC1" gate="G$1" pin="PB2(SS/OC1B)"/>
+<wire x1="76.2" y1="-58.42" x2="81.28" y2="-58.42" width="0.1524" layer="91"/>
+<label x="81.28" y="-58.42" size="1.778" layer="95"/>
 </segment>
 </net>
@@
 <label x="-38.1" y="-182.88" size="1.778" layer="95"/>
 </segment>
+<segment>
+<pinref part="IC1" gate="G$1" pin="PC1(ADC1)"/>
+<wire x1="76.2" y1="-10.16" x2="81.28" y2="-10.16" width="0.1524" layer="91"/>
+<label x="81.28" y="-10.16" size="1.778" layer="95"/>
+</segment>
 </net>
 <net name="BTN_2" class="0">
@@
 <label x="-25.4" y="-182.88" size="1.778" layer="95"/>
 </segment>
-</net>
-<net name="BTN_3" class="0">
-<segment>
-<pinref part="R9" gate="G$1" pin="1"/>
-<pinref part="U$5" gate="G$1" pin="4"/>
-<wire x1="-17.78" y1="-162.56" x2="-17.78" y2="-160.02" width="0.1524" layer="91"/>
-<wire x1="-17.78" y1="-160.02" x2="-12.7" y2="-160.02" width="0.1524" layer="91"/>
-<wire x1="-12.7" y1="-160.02" x2="-12.7" y2="-182.88" width="0.1524" layer="91"/>
-<junction x="-17.78" y="-160.02"/>
-<label x="-12.7" y="-182.88" size="1.778" layer="95"/>
-</segment>
-</net>
+<segment>
+<pinref part="IC1" gate="G$1" pin="PC2(ADC2)"/>
+<wire x1="76.2" y1="-12.7" x2="81.28" y2="-12.7" width="0.1524" layer="91"/>
+<label x="81.28" y="-12.7" size="1.778" layer="95"/>
+</segment>
+</net>
+<net name="N$14" class="0">
+<segment>
+<pinref part="U$2" gate="G$1" pin="VBAT"/>
+<wire x1="152.4" y1="-17.78" x2="167.64" y2="-17.78" width="0.1524" layer="91"/>
+<wire x1="167.64" y1="-17.78" x2="167.64" y2="-30.48" width="0.1524" layer="91"/>
+<pinref part="B1" gate="2477" pin="+"/>
+</segment>
+</net>

Commit message: PCB v1
Parts:
- added C6, C7, C8: 10uF, SparkFun-Capacitors:10UF-16V-10%(TANT)
- added R9: 4.7k, resistor:R-EU_R0805
- C1, C2, C3, C4, C5: value (none) -> 0.1
- R1, R2, R4, R5, R6, R8: value (none) -> 4.7k
- R3: value (none) -> 10k
- R7: value (none) -> 68k
Connections:
- new net USB_D+: U$8.D+
- new net USB_D-: U$8.D-
- net GND: now also C6.-, C7.-, U$8.GND
- net PHOTO_SENSOR: now also C8.-
- net RESET: now also R9.1
- net VCC: now also C6.+, C7.+, C8.+, R9.2, U$8.VCC

Commit message: PCB design
Parts:
- removed C3: 0.1, resistor:C-EUC0805
- removed C7: 10uF, SparkFun-Capacitors:10UF-16V-10%(TANT)
Connections:
- net GND: no longer C3.2, C7.-
- net VCC: no longer C3.1, C7.+
Other:
- moved on the sheet: B1, C1, C2, C4, C5, C6, C8, IC1, R1, R2, R3, R4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

Commit message: .
Parts:
- removed C1, C2, C4: 0.1, resistor:C-EUC0805
- removed C6: 10uF, SparkFun-Capacitors:10UF-16V-10%(TANT)
- removed IC1: MEGA8-AI, atmel:MEGA8-AI
- removed R6, R8: 4.7k, resistor:R-EU_R0805
- removed U$3, U$4: IT1188E, misc:IT1188E
- removed U$9: PINHD-1X5, PLL:PINHD-1X5
- added U1: (no value), esp8266modules:ESP12ESMD
Connections:
- removed net BTN_1: IC1.PC1(ADC1), R6.1, U$3.4
- removed net BTN_2: IC1.PC2(ADC2), R8.1, U$4.4
- removed net MISO: IC1.PB4(MISO), U$9.2
- removed net MOSI: IC1.PB3(MOSI/OC2), U$9.1
- removed net SCK: IC1.PB5(SCK), U$9.3
- removed net VCC: C1.1, C2.1, C4.1, C6.+, C8.+, IC1.AREF, IC1.AVCC, IC1.VCC@1, IC1.VCC@2, R1.2, R2.2, R3.1, R4.2, R5.2, R6.2, R8.2, R9.2, U$2.VCC, U$6.P$2, U$7.VCC, U$8.VCC
- new net +3V3: C8.+, R1.2, R2.2, R4.2, R5.2, R9.2, U$2.VCC, U$6.P$2, U1.VCC
- new net +5V: R3.1, U$7.VCC, U$8.VCC
- new net RX: U1.RX
- new net TX: U1.TX
- net DSP_CLK: no longer IC1.PB0(ICP)
- net DSP_DIN: no longer IC1.PB2(SS/OC1B)
- net DSP_LOAD: no longer IC1.PB1(OC1A)
- net GND: now also U1.GND; no longer C1.2, C2.2, C4.2, C6.-, IC1.GND, IC1.GND@1, IC1.GND@2, U$3.3, U$4.3, U$9.5
- net PHOTO_SENSOR: now also U1.ADC; no longer IC1.PC0(ADC0)
- net RESET: now also U1.RESET; no longer IC1.PC6(/RESET), U$9.4
- net SCL: no longer IC1.PC5(ADC5/SCL)
- net SDA: no longer IC1.PC4(ADC4/SDA)
- net SQW: no longer IC1.PD2(INT0)
- net TIMER_INT: no longer IC1.PD3(INT1)
